File: Hardware/AddaTone MAX5134 DAC.sch (KiCad schematic (older format))
At the start: 97 parts, among them J1 SWD_Header, J2 PItch_In, J3 PD1_Amt_In, J4 PD2_Amt_In, J5 VCA_In, J6 DAC1_Out, J7 DAC2_Out, J8 Eurorack_16_pin_power, SW1 SW_SPST, SW2 SW_SPST, SW3 SW_SPST, SW4 SW_SPST, U1 STM32F446RETx, U2 ICE40UP5K-SG48ITR, U3 MCP6004, U5 TL072, U6 LD1117S12TR_SOT223, U7 LM1117-3.3, Y1 ECS-12MHz

Commit message: Updated schematic for PCM5100 DAC
Parts:
- removed C? (x2): 2.2uF, symbol Device:C
- removed C? (x4): 100nF, symbol Device:C
- removed C? (x2): 10uF, symbol Device:C
- removed C?: 1nF, Capacitors_SMD:C_0805_HandSoldering, symbol Device:C
- removed C?: 100pF, Capacitors_SMD:C_0805_HandSoldering, symbol Device:C
- removed R?: 1k, Resistors_SMD:R_0805_HandSoldering, symbol Device:R
- removed R?: 33k, Resistors_SMD:R_0805_HandSoldering, symbol Device:R
- removed R?: 2.2k, Resistors_SMD:R_0805_HandSoldering, symbol Device:R
- removed R?: 10k, Resistors_SMD:R_0805_HandSoldering, symbol Device:R
- removed U?: PCM5100APW, Package_SO:TSSOP-20_4.4x6.5mm_P0.65mm, symbol PCM5100APW:PCM5100APW
- removed U?: TL072, SMD_Packages:SOIC-8-N, symbol Amplifier_Operational:TL072
- added C31: 100nF, Capacitors_SMD:C_0805_HandSoldering, symbol Device:C
- added C33: 10uF, Capacitors_SMD:C_0805_HandSoldering, symbol Device:C
- added C35: 18pF, Capacitors_SMD:C_0805_HandSoldering, symbol Device:C
- added R15: 47k, Resistors_SMD:R_0805_HandSoldering, symbol Device:R
- added R17: 6.8k, Resistors_SMD:R_0805_HandSoldering, symbol Device:R
- added R19: 39k, Resistors_SMD:R_0805_HandSoldering, symbol Device:R
- added R21: 1k, Resistors_SMD:R_0805_HandSoldering, symbol Device:R
- added U4: MAX5134, Housings_SSOP:TSSOP-16_4.4x5mm_Pitch0.65mm, symbol MAX5134:MAX5134
- added unit 2 of U5
- C32: value 1nF -> 10uF
- C34: value 100pF -> 18pF
- R14: value 2.2k -> 47k
- R16: value 10k -> 6.8k
- R18: value 33k -> 39k
Connections:
- net labels added: DAC_CLK, DAC_MOSI, DAC_~CS
- net labels removed: DAC_BCLK, DAC_DATA, DAC_LRCLK
- wire segments 376 -> 354
- no-connect marks 56 -> 59
Other:
- note added: "Switches"
- moved on the sheet: C32, C36, C37, C38, C41, C42, D2, L1, R14, R22, SW1, SW2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
