File: Hardware/AddaTone Controls.kicad_pcb (KiCad board)
At the start: 2 copper layers, 60 x 110 mm, 18 parts, among them J1 Conn_01x10_Male, J2 Conn_01x12_Male, J3 Pitch_In, J4 Harm1_In, J5 Harm2_In, J6 Warp_In, J7 DAC1_Out, J8 DAC2_Out, SW1 SW_Push, SW2 SW_Push, SW3 SW_SPST, SW4 SW_SPST

Commit message: Updates to PCB layout
Other:
- board text added: "Addatone Controls v1.0"
Changed lines of the file:
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@@
   (general
     (thickness 1.6)
-    (drawings 48)
+    (drawings 49)
     (tracks 144)
     (zones 0)
@@
   (page A4)
   (layers
-    (0 F.Cu signal hide)
-    (31 B.Cu signal hide)
-    (32 B.Adhes user)
+    (0 F.Cu signal)
+    (31 B.Cu signal)
+    (32 B.Adhes user hide)
     (33 F.Adhes user hide)
     (34 B.Paste user)
@@
     (38 B.Mask user)
     (39 F.Mask user)
-    (40 Dwgs.User user)
-    (41 Cmts.User user)
-    (42 Eco1.User user)
-    (43 Eco2.User user)
+    (40 Dwgs.User user hide)
+    (41 Cmts.User user hide)
+    (42 Eco1.User user hide)
+    (43 Eco2.User user hide)
     (44 Edge.Cuts user)
-    (45 Margin user)
+    (45 Margin user hide)
     (46 B.CrtYd user)
     (47 F.CrtYd user)
@@
       (drillshape 0)
       (scaleselection 1)
-      (outputdirectory "Gerbers/PCB/"))
+      (outputdirectory "Gerbers/Controls/"))
   )
   (net 0 "")
@@
       (rotate (xyz 0 0 0))
     )
+  )
+  (gr_text "Addatone Controls v1.0" (at 131.1 54.2) (layer B.SilkS)
+    (effects (font (size 1.5 1.5) (thickness 0.3)) (justify mirror))
   )
   (gr_text Mix (at 150 91) (layer B.SilkS)
@@
   (segment (start 114.773998 113.2) (end 146 81.973998) (width 0.5) (layer F.Cu) (net 13))
   (segment (start 106.6 113.2) (end 114.773998 113.2) (width 0.5) (layer F.Cu) (net 13))
-  (segment (start 149.5 92.7) (end 144.073998 92.7) (width 0.5) (layer F.Cu) (net 22))
-  (segment (start 130 106.773998) (end 130 113) (width 0.5) (layer F.Cu) (net 22))
-  (via (at 149.5 92.7) (size 0.8) (drill 0.4) (layers F.Cu B.Cu) (net 22))
-  (segment (start 144.073998 92.7) (end 130 106.773998) (width 0.5) (layer F.Cu) (net 22))
-  (segment (start 149.5 92.7) (end 155.5 92.7) (width 0.5) (layer B.Cu) (net 22))
-  (segment (start 107.8 118.526002) (end 107.8 116.6) (width 0.5) (layer F.Cu) (net 21))
-  (segment (start 125.5 146.08) (end 125.5 136.226002) (width 0.5) (layer F.Cu) (net 21))
-  (via (at 107.8 116.6) (size 0.8) (drill 0.4) (layers F.Cu B.Cu) (net 21))
-  (segment (start 125.5 136.226002) (end 107.8 118.526002) (width 0.5) (layer F.Cu) (net 21))
-  (segment (start 107.8 109.84) (end 102.8 104.84) (width 0.5) (layer B.Cu) (net 21))
-  (segment (start 107.8 116.6) (end 107.8 109.84) (width 0.5) (layer B.Cu) (net 21))
   (via (at 118.3 101.1) (size 0.8) (drill 0.4) (layers F.Cu B.Cu) (net 14))
   (segment (start 123.050001 140.779999) (end 123.050001 105.850001) (width 0.5) (layer B.Cu) (net 14))
@@
   (segment (start 116.226002 109.92) (end 130 96.146002) (width 0.5) (layer F.Cu) (net 17))
   (segment (start 102.8 109.92) (end 116.226002 109.92) (width 0.5) (layer F.Cu) (net 17))
+  (segment (start 107.8 118.526002) (end 107.8 116.6) (width 0.5) (layer F.Cu) (net 21))
+  (segment (start 125.5 146.08) (end 125.5 136.226002) (width 0.5) (layer F.Cu) (net 21))
+  (via (at 107.8 116.6) (size 0.8) (drill 0.4) (layers F.Cu B.Cu) (net 21))
+  (segment (start 125.5 136.226002) (end 107.8 118.526002) (width 0.5) (layer F.Cu) (net 21))
+  (segment (start 107.8 109.84) (end 102.8 104.84) (width 0.5) (layer B.Cu) (net 21))
+  (segment (start 107.8 116.6) (end 107.8 109.84) (width 0.5) (layer B.Cu) (net 21))
+  (segment (start 149.5 92.7) (end 144.073998 92.7) (width 0.5) (layer F.Cu) (net 22))
+  (segment (start 130 106.773998) (end 130 113) (width 0.5) (layer F.Cu) (net 22))
+  (via (at 149.5 92.7) (size 0.8) (drill 0.4) (layers F.Cu B.Cu) (net 22))
+  (segment (start 144.073998 92.7) (end 130 106.773998) (width 0.5) (layer F.Cu) (net 22))
+  (segment (start 149.5 92.7) (end 155.5 92.7) (width 0.5) (layer B.Cu) (net 22))
   (zone (net 1) (net_name GND) (layer B.Cu) (hatch edge 0.508)
     (connect_pads (clearance 0.508))

Commit message: Updated pcb files to Kicad 6.0
Other:
- net class Default removed
- net class Wide_Power removed
