File: Hardware/AddaTone components.kicad_sch (KiCad schematic)
At the start: 95 parts, among them J1 SWD_Header, J2 Conn_01x10_Female, J3 Conn_01x12_Female, J4 Conn_01x03_Male, J5 Conn_01x06_Male, J6 Conn_01x03_Male, J7 Conn_01x02_Male, J8 Eurorack_16_pin_power, U1 STM32F446RETx, U2 ICE40UP5K-SG48ITR, U3 MCP6004, U4 PCM5100APW, U5 TL072, U6 LD1117S12TR, U7 LM1117-3.3, Y1 ECS-12MHz

Commit message: Updated schematic and pcb to v2.1
Parts:
- removed R23: 0, Jumper:SolderJumper-2_P1.3mm_Bridged_Pad1.0x1.5mm, symbol Device:R
- added JP1: Jumper_2_Bridged, Jumper:SolderJumper-2_P1.3mm_Bridged_Pad1.0x1.5mm, symbol Jumper:Jumper_2_Bridged
- C1, C10, C11, C12, C13, C14, C15, C16, C17, C18, C19, C2, C20, C21, C22, C23, C24, C25, C26, C27, C28, C29, C3, C30, C31, C32, C33, C34, C35, C36, C37, C38, C4, C41, C42, C43, C5, C6, C7, C8, C9: symbol Device:C -> Device:C_Small
- C39, C40: symbol AddaTone components-rescue:CP-Device -> Device:C_Polarized_Small
- R1, R10, R11, R12, R13, R14, R15, R16, R17, R18, R19, R2, R20, R21, R22, R24, R3, R4, R5, R6, R7, R8, R9: symbol Device:R -> Device:R_Small
Connections:
- net +3V3: now also JP1.2 (B)
- net FPGA_3V3: now also JP1.1 (A)
Other:
- note added: "Connectors"
- note added: "DAC"
- note added: "FPGA"
- note added: "Microcontroller"
- note added: "Test Points"
- moved on the sheet: C1, C10, C11, C12, C13, C14, C15, C16, C17, C18, C19, C2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
